Commit message: URDF moved in a correct place My polar IK fixed

File: GUI/urdf/braccio.urdf (robot description, URDF)
Before this commit: robot visual, 9 links, 8 joints
Links:
- link gripper_base: geometry visual mesh filename=gripper_base.stl
- link gripper_fix: geometry visual mesh filename=gripper_fix.stl
- link gripper_movable: geometry visual mesh filename=gripper_movable.stl
- link link1: geometry visual mesh filename=base.stl
- link link2: geometry visual mesh filename=shoulder.stl
- link link3: geometry visual mesh filename=elbow.stl
- link link4: geometry visual mesh filename=wrist_pitch.stl
- link link5: geometry visual mesh filename=wrist_roll.stl
